File: hardware/kicad/novapcb-layout-v1.1/novapcb-layout-v1.1.kicad_pcb (KiCad board)
At the start: 6 copper layers, 90 x 70 mm, 129 parts, among them J1 USB-C_2.0, J10 CRSF_solder_pad, J11 ESC_solder_pad, J12 ESC_solder_pad, J13 ESC_solder_pad, J14 ESC_solder_pad, J15 ESC_solder_pad, J16 ESC_solder_pad, J17 ESC_solder_pad, J18 ESC_solder_pad, J19 MAUCH2_6P, J2 microSD_DM3AT, J20 CAN_4P, J3 TELEM_6P, J4 MAUCH_6P, J5 GPS_MAG_10P, J9 SWD_10P, Q2 AO3401A, Q3 AO4262E, Q4 AO4262E, Q5 AO3400A, U1 STM32H743VITx, U11 LM74700-Q1, U12 LM74700-Q1, U13 LP5907MFX-3.3, U14 TJA1051TK/3, U15 PESD2CAN, U2 AP2112K-3.3, U3 ICM-42688-P_LGA-14_2.5x3mm_P0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, U4 DPS310, U5 USBLC6-2P6, U6 TPS25940A, U7 LPS22HB, U8 BMI088, U9 LSM6DSV16X, Y1 8MHz

Commit message: hw: R4 placement GENUINELY CLEAN — 0 DRC + valid slot (master 2026-05-22)
153 (v4) → 18 (v12 false-0) → 1 → 0 via:
1. Slot: single 13-vertex closed polygon defining ONLY the 2mm kerf
   (not the U-shaped REGION). Island has board material under sensors.
2. Heater cluster (Q5/R61/U13/FB2) un-pinned — greedy places them via
   ideal-pos + spiral.
3. R31/R32 USB-CC pull-down resistors pinned clear of J1 USB-C.
4. R45/R46 CAN termination pinned south of U14 (74,21)/(78,21) with
   4mm X separation to clear courtyards.
5. ESC pad keepout extended to Y=2..9 X=±9 from each ESC cluster
   center — decoupling caps stay clear of ESC pad rows.

Final state:
- 0 DRC violations ✓
- 76/76 smalls placed ✓
- Slot properly thin U-kerf with bridge ✓
- All sensors on board material (verified via render_clean_v13_island.png)
- 235 unconnected (expected — no routes yet)

Renders:
- render_clean_v13_top.png + bot.png — full board
- render_clean_v13_island.png — zoomed S-island F.Cu + B.Cu

Per master "DRC alone is NOT sufficient verification" — visual
verification confirmed via island zoom render.

Co-Authored-By: Claude Opus 4.7 <noreply@anthropic.com>
Parts:
- moved C77 11.4 mm to (72.4, 50.3)
- moved C32 9.77 mm to (78.9, 5.41)
- moved R61 8.99 mm to (65.9, 55.7)
- moved C9 8.94 mm to (76.7, 14.7)
- moved C96 7.07 mm to (46.0, 55.6)
- moved Q5 6.82 mm to (59.8, 55.2)
- moved R31 5.92 mm to (73.0, 31.5)
- moved R32 5.92 mm to (73.0, 28.5)
- moved R45 5.63 mm to (74.0, 21.0)
- moved R22 4.20 mm to (54.8, 60.0)
- moved C92 3.91 mm to (46.5, 60.0)
- moved R46 3.42 mm to (78.0, 21.0)
- moved R21 2.92 mm to (57.1, 59.9)
- moved C93 2.87 mm to (46.5, 57.1)
- moved FB2 2.83 mm to (60.0, 60.0)
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Changed lines of the file:
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@@
 	(footprint "Capacitor_SMD:C_0402_1005Metric"
 		(layer "F.Cu")
-		(at 43 54.58)
+		(at 43 54.33)
 		(descr "Capacitor SMD 0402 (1005 Metric), square (rectangular) end terminal, IPC-7351 nominal, (Body size source: IPC-SM-782 page 76, https://www.pcb-3d.com/wordpress/wp-content/uploads/ipc-sm-782a_amendment_1_and_2.pdf), generated with kicad-footprint-generator")
 		(tags "capacitor")
@@
 	(footprint "Capacitor_SMD:C_0402_1005Metric"
 		(layer "F.Cu")
-		(at 40.171572 55.751572)
+		(at 39.994796 55.574796)
 		(descr "Capacitor SMD 0402 (1005 Metric), square (rectangular) end terminal, IPC-7351 nominal, (Body size source: IPC-SM-782 page 76, https://www.pcb-3d.com/wordpress/wp-content/uploads/ipc-sm-782a_amendment_1_and_2.pdf), generated with kicad-footprint-generator")
 		(tags "capacitor")
@@
 	(footprint "Resistor_SMD:R_0603_1608Metric"
 		(layer "F.Cu")
-		(at 79.531278 22.072391)
+		(at 74 21)
 		(descr "Resistor SMD 0603 (1608 Metric), square (rectangular) end terminal, IPC-7351 nominal, (Body size source: IPC-SM-782 page 72, https://www.pcb-3d.com/wordpress/wp-content/uploads/ipc-sm-782a_amendment_1_and_2.pdf), generated with kicad-footprint-generator")
 		(tags "resistor")
@@
 	(footprint "Resistor_SMD:R_0603_1608Metric"
 		(layer "F.Cu")
-		(at 75.355602 23.161582)
+		(at 78 21)
 		(descr "Resistor SMD 0603 (1608 Metric), square (rectangular) end terminal, IPC-7351 nominal, (Body size source: IPC-SM-782 page 72, https://www.pcb-3d.com/wordpress/wp-content/uploads/ipc-sm-782a_amendment_1_and_2.pdf), generated with kicad-footprint-generator")
 		(tags "resistor")
@@
 	(footprint "Capacitor_SMD:C_0805_2012Metric"
 		(layer "F.Cu")
-		(at 69.312692 7.44957)
+		(at 78.86764 5.407359)
 		(descr "Capacitor SMD 0805 (2012 Metric), square (rectangular) end terminal, IPC-7351 nominal, (Body size source: IPC-SM-782 page 76, https://www.pcb-3d.com/wordpress/wp-content/uploads/ipc-sm-782a_amendment_1_and_2.pdf, https://docs.google.com/spreadsheets/d/1BsfQQcO9C6DZCsRaXUlFlo91Tg2WpOkGARC1WS5S8t0/edit?usp=sharing), generated with kicad-footprint-generator")
 		(tags "capacitor")
@@
 	(footprint "Capacitor_SMD:C_0402_1005Metric"
 		(layer "F.Cu")
-		(at 45.298097 56.281902)
+		(at 46.464548 60.015062)
 		(descr "Capacitor SMD 0402 (1005 Metric), square (rectangular) end terminal, IPC-7351 nominal, (Body size source: IPC-SM-782 page 76, https://www.pcb-3d.com/wordpress/wp-content/uploads/ipc-sm-782a_amendment_1_and_2.pdf), generated with kicad-footprint-generator")
 		(tags "capacitor")
@@
 	(footprint "Resistor_SMD:R_0402_1005Metric"
 		(layer "F.Cu")
-		(at 55.87 55.94)
+		(at 54.809339 60.00066)
 		(descr "Resistor SMD 0402 (1005 Metric), square (rectangular) end terminal, IPC-7351 nominal, (Body size source: IPC-SM-782 page 72, https://www.pcb-3d.com/wordpress/wp-content/uploads/ipc-sm-782a_amendment_1_and_2.pdf), generated with kicad-footprint-generator")
 		(tags "resistor")
@@
 	(footprint "Resistor_SMD:R_0402_1005Metric"
 		(layer "F.Cu")
-		(at 78.905 28.95)
+		(at 73 28.5)
 		(descr "Resistor SMD 0402 (1005 Metric), square (rectangular) end terminal, IPC-7351 nominal, (Body size source: IPC-SM-782 page 72, https://www.pcb-3d.com/wordpress/wp-content/uploads/ipc-sm-782a_amendment_1_and_2.pdf), generated with kicad-footprint-generator")
 		(tags "resistor")
@@
 	(footprint "Capacitor_SMD:C_0402_1005Metric"
 		(layer "F.Cu")
-		(at 46.464548 60.015062)
+		(at 46.464548 57.144937)
 		(descr "Capacitor SMD 0402 (1005 Metric), square (rectangular) end terminal, IPC-7351 nominal, (Body size source: IPC-SM-782 page 76, https://www.pcb-3d.com/wordpress/wp-content/uploads/ipc-sm-782a_amendment_1_and_2.pdf), generated with kicad-footprint-generator")
 		(tags "capacitor")
@@
 	(footprint "Capacitor_SMD:C_0402_1005Metric"
 		(layer "F.Cu")
-		(at 62.985 56.75)
+		(at 72.404329 50.26903)
 		(descr "Capacitor SMD 0402 (1005 Metric), square (rectangular) end terminal, IPC-7351 nominal, (Body size source: IPC-SM-782 page 76, https://www.pcb-3d.com/wordpress/wp-content/uploads/ipc-sm-782a_amendment_1_and_2.pdf), generated with kicad-footprint-generator")
 		(tags "capacitor")
@@
 	(footprint "Resistor_SMD:R_0402_1005Metric"
 		(layer "F.Cu")
-		(at 78.905 31.95)
+		(at 73 31.5)
 		(descr "Resistor SMD 0402 (1005 Metric), square (rectangular) end terminal, IPC-7351 nominal, (Body size source: IPC-SM-782 page 72, https://www.pcb-3d.com/wordpress/wp-content/uploads/ipc-sm-782a_amendment_1_and_2.pdf), generated with kicad-footprint-generator")
 		(tags "resistor")
@@
 	(footprint "Capacitor_SMD:C_0402_1005Metric"
 		(layer "F.Cu")
-		(at 45.540668 57.52762)
+		(at 46.5 58.58)
 		(descr "Capacitor SMD 0402 (1005 Metric), square (rectangular) end terminal, IPC-7351 nominal, (Body size source: IPC-SM-782 page 76, https://www.pcb-3d.com/wordpress/wp-content/uploads/ipc-sm-782a_amendment_1_and_2.pdf), generated with kicad-footprint-generator")
 		(tags "capacitor")
@@
 	(footprint "Inductor_SMD:L_0402_1005Metric"
 		(layer "F.Cu")
-		(at 62 58)
+		(at 60 60)
 		(descr "Inductor SMD 0402 (1005 Metric), square (rectangular) end terminal, IPC-7351 nominal, (Body size source: http://www.tortai-tech.com/upload/download/2011102023233369053.pdf), generated with kicad-footprint-generator")
 		(tags "inductor")
@@
 	(footprint "Capacitor_SMD:C_0402_1005Metric"
 		(layer "F.Cu")
-		(at 39.073511 56.953595)
+		(at 46.005203 55.574796)
 		(descr "Capacitor SMD 0402 (1005 Metric), square (rectangular) end terminal, IPC-7351 nominal, (Body size source: IPC-SM-782 page 76, https://www.pcb-3d.com/wordpress/wp-content/uploads/ipc-sm-782a_amendment_1_and_2.pdf), generated with kicad-footprint-generator")
 		(tags "capacitor")
@@
 	(footprint "Capacitor_SMD:C_0402_1005Metric"
 		(layer "F.Cu")
-		(at 43 55.83)
+		(at 43 55.58)
 		(descr "Capacitor SMD 0402 (1005 Metric), square (rectangular) end terminal, IPC-7351 nominal, (Body size source: IPC-SM-782 page 76, https://www.pcb-3d.com/wordpress/wp-content/uploads/ipc-sm-782a_amendment_1_and_2.pdf), generated with kicad-footprint-generator")
 		(tags "capacitor")
@@
 	(footprint "Resistor_SMD:R_0402_1005Metric"
 		(layer "F.Cu")
-		(at 56.7 62.78)
+		(at 57.053553 59.883553)
 		(descr "Resistor SMD 0402 (1005 Metric), square (rectangular) end terminal, IPC-7351 nominal, (Body size source: IPC-SM-782 page 72, https://www.pcb-3d.com/wordpress/wp-content/uploads/ipc-sm-782a_amendment_1_and_2.pdf), generated with kicad-footprint-generator")
 		(tags "resistor")
@@
 	(footprint "Capacitor_SMD:C_0402_1005Metric"
 		(layer "F.Cu")
-		(at 78.33731 5.937689)
+		(at 76.729758 14.731337)
 		(descr "Capacitor SMD 0402 (1005 Metric), square (rectangular) end terminal, IPC-7351 nominal, (Body size source: IPC-SM-782 page 76, https://www.pcb-3d.com/wordpress/wp-content/uploads/ipc-sm-782a_amendment_1_and_2.pdf), generated with kicad-footprint-generator")
 		(tags "capacitor")
@@
 	(footprint "Resistor_SMD:R_2512_6332Metric"
 		(layer "F.Cu")
-		(at 58 60)
+		(at 65.88321 55.669696)
 		(descr "Resistor SMD 2512 (6332 Metric), square (rectangular) end terminal, IPC-7351 nominal, (Body size source: IPC-SM-782 page 72, https://www.pcb-3d.com/wordpress/wp-content/uploads/ipc-sm-782a_amendment_1_and_2.pdf), generated with kicad-footprint-generator")
 		(tags "resistor")
@@
 	(footprint "Package_TO_SOT_SMD:SOT-23"
 		(layer "F.Cu")
-		(at 55 60)
+		(at 59.823223 55.176776)
 		(descr "SOT, 3 Pin (JEDEC TO-236 Var AB https://www.jedec.org/document_search?search_api_views_fulltext=TO-236), generated with kicad-footprint-generator ipc_gullwing_generator.py")
 		(tags "SOT TO_SOT_SMD")
@@
 	(footprint "Connector_PinHeader_1.27mm:PinHeader_2x05_P1.27mm_Vertical_SMD"
 		(layer "B.Cu")
-		(at 41 62)
+		(at 41 60)
 		(descr "surface-mounted straight pin header, 2x05, 1.27mm pitch, double rows")
 		(tags "Surface mounted pin header SMD 2x05 1.27mm double row")
@@
 	)
 	(gr_line
-		(start 52 51)
-		(end 72 51)
+		(start 70 65)
+		(end 70 53)
 		(stroke
 			(width 0.1)
@@
 	)
 	(gr_line
-		(start 27 53)
-		(end 27 65)
+		(start 70 53)
+		(end 52 53)
 		(stroke
 			(width 0.1)
@@
 		(layer "Edge.Cuts")
 	)
-	(gr_line
-		(start 25 51)
-		(end 38 51)
+	(gr_rect
+		(start 0 0)
+		(end 90 70)
 		(stroke
-			(width 0.1)
+			(width 0.15)
 			(type default)
 		)
+		(fill no)
 		(layer "Edge.Cuts")
 	)
 	(gr_line
-		(start 27 65)
-		(end 70 65)
+		(start 27 53)
+		(end 27 65)
 		(stroke
 			(width 0.1)
@@
 		(layer "Edge.Cuts")
 	)
-	(gr_rect
-		(start 0 0)
-		(end 90 70)
+	(gr_line
+		(start 25 51)
+		(end 38 51)
 		(stroke
-			(width 0.15)
+			(width 0.1)
 			(type default)
 		)
-		(fill no)
 		(layer "Edge.Cuts")
 	)
 	(gr_line
-		(start 25 67)
-		(end 25 51)
+		(start 38 53)
+		(end 27 53)
 		(stroke
 			(width 0.1)
@@
 	)
 	(gr_line
-		(start 70 65)
-		(end 70 53)
+		(start 25 67)
+		(end 25 51)
 		(stroke
 			(width 0.1)
@@
 	)
 	(gr_line
-		(start 70 53)
-		(end 52 53)
+		(start 27 65)
+		(end 70 65)
 		(stroke
 			(width 0.1)
@@
 	)
 	(gr_line
-		(start 38 53)
-		(end 27 53)
+		(start 38 51)
+		(end 38 53)
 		(stroke
 			(width 0.1)
@@
 	)
 	(gr_line
-		(start 38 51)
-		(end 38 53)
+		(start 52 53)
+		(end 52 51)
 		(stroke
 			(width 0.1)
@@
 	)
 	(gr_line
-		(start 52 53)
-		(end 52 51)
+		(start 52 51)
+		(end 72 51)
 		(stroke
 			(width 0.1)

Commit message: hw: R4 PCB-level pin re-mux on U1 (master 2026-05-22)
16 pad-net swaps on U1 to enact the placement strategy re-mux:
- SPI1_MOSI: pin 88 (N) → pin 31 (PA7 S, was HEATER_PWM)
- SPI3 SCK/MISO/MOSI: pins 89/90/91 (N) → pins 28/32/33 (S)
- I2C1 SCL/SDA: pins 92/93 (N) → pins 36/37 (S)
- GPS1 TX/RX: pins 86/87 (N) → pins 57/58 (E)
- 8× MOT: scattered (S/W/E) → all to N (pins 86-95)

HEATER_PWM lands at pin 88 (N side) — needs timer-capable AF
verification before tape-out (deferred).

Re-mux done at PCB level (pad-net swap) — project has no .kicad_sch
files so schematic edit + ERC are not possible in this session.
Master's "verify EVERY AF against DS12110 Table 11 LQFP-100 column"
is the proper follow-up requiring datasheet access; the routing
test validates the net topology only.

Pin counts per side AFTER re-mux:
  N=22 (was 21)  E=18 (was 18)  S=16 (was 13)  W=17 (was 21)
All sides comfortably under 25.

Now running Freerouting -mp 30 v2.2.3 on the re-muxed PCB. The gate:
must reach ~100% or honest plateau report.

Co-Authored-By: Claude Opus 4.7 <noreply@anthropic.com>
Connections:
- U1 pad 22: MOT3 -> (no net)
- U1 pad 23: MOT4 -> (no net)
- U1 pad 24: MOT5 -> (no net)
- U1 pad 25: MOT6 -> (no net)
- U1 pad 28: (no net) -> SPI3_SCK
- U1 pad 31: HEATER_PWM -> SPI1_MOSI
- U1 pad 32: (no net) -> SPI3_MISO
- U1 pad 33: (no net) -> SPI3_MOSI
- U1 pad 34: MOT1 -> (no net)
- U1 pad 35: MOT2 -> (no net)
- U1 pad 36: (no net) -> I2C1_SCL
- U1 pad 37: (no net) -> I2C1_SDA
- U1 pad 57: (no net) -> GPS1_TX
- U1 pad 58: (no net) -> GPS1_RX
- U1 pad 59: MOT7 -> (no net)
- U1 pad 60: MOT8 -> (no net)
- U1 pad 86: GPS1_TX -> MOT1
- U1 pad 87: GPS1_RX -> MOT2
- U1 pad 88: SPI1_MOSI -> HEATER_PWM
- U1 pad 89: SPI3_SCK -> MOT3
- U1 pad 90: SPI3_MISO -> MOT4
- U1 pad 91: SPI3_MOSI -> MOT5
- U1 pad 92: I2C1_SCL -> MOT6
- U1 pad 93: I2C1_SDA -> MOT7
- U1 pad 95: (no net) -> MOT8
Changed lines of the file:
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@@
 			(layers "F.Cu" "F.Mask" "F.Paste")
 			(roundrect_rratio 0.25)
-			(net 57 "MOT3")
 		)
 		(pad "23" smd roundrect
@@
 			(layers "F.Cu" "F.Mask" "F.Paste")
 			(roundrect_rratio 0.25)
-			(net 58 "MOT4")
 		)
 		(pad "24" smd roundrect
@@
 			(layers "F.Cu" "F.Mask" "F.Paste")
 			(roundrect_rratio 0.25)
-			(net 59 "MOT5")
 		)
 		(pad "25" smd roundrect
@@
 			(layers "F.Cu" "F.Mask" "F.Paste")
 			(roundrect_rratio 0.25)
-			(net 60 "MOT6")
 		)
 		(pad "26" smd roundrect
@@
 			(layers "F.Cu" "F.Mask" "F.Paste")
 			(roundrect_rratio 0.25)
+			(net 84 "SPI3_SCK")
 		)
 		(pad "29" smd roundrect
@@
 			(layers "F.Cu" "F.Mask" "F.Paste")
 			(roundrect_rratio 0.25)
-			(net 34 "HEATER_PWM")
+			(net 77 "SPI1_MOSI")
 		)
 		(pad "32" smd roundrect
@@
 			(layers "F.Cu" "F.Mask" "F.Paste")
 			(roundrect_rratio 0.25)
+			(net 82 "SPI3_MISO")
 		)
 		(pad "33" smd roundrect
@@
 			(layers "F.Cu" "F.Mask" "F.Paste")
 			(roundrect_rratio 0.25)
+			(net 83 "SPI3_MOSI")
 		)
 		(pad "34" smd roundrect
@@
 			(layers "F.Cu" "F.Mask" "F.Paste")
 			(roundrect_rratio 0.25)
-			(net 55 "MOT1")
 		)
 		(pad "35" smd roundrect
@@
 			(layers "F.Cu" "F.Mask" "F.Paste")
 			(roundrect_rratio 0.25)
-			(net 56 "MOT2")
 		)
 		(pad "36" smd roundrect
@@
 			(layers "F.Cu" "F.Mask" "F.Paste")
 			(roundrect_rratio 0.25)
+			(net 37 "I2C1_SCL")
 		)
 		(pad "37" smd roundrect
@@
 			(layers "F.Cu" "F.Mask" "F.Paste")
 			(roundrect_rratio 0.25)
+			(net 38 "I2C1_SDA")
 		)
 		(pad "38" smd roundrect
@@
 			(layers "F.Cu" "F.Mask" "F.Paste")
 			(roundrect_rratio 0.25)
+			(net 32 "GPS1_TX")
 		)
 		(pad "58" smd roundrect
@@
 			(layers "F.Cu" "F.Mask" "F.Paste")
 			(roundrect_rratio 0.25)
+			(net 31 "GPS1_RX")
 		)
 		(pad "59" smd roundrect
@@
 			(layers "F.Cu" "F.Mask" "F.Paste")
 			(roundrect_rratio 0.25)
-			(net 61 "MOT7")
 		)
 		(pad "60" smd roundrect
@@
 			(layers "F.Cu" "F.Mask" "F.Paste")
 			(roundrect_rratio 0.25)
-			(net 62 "MOT8")
 		)
 		(pad "61" smd roundrect
@@
 			(layers "F.Cu" "F.Mask" "F.Paste")
 			(roundrect_rratio 0.25)
-			(net 32 "GPS1_TX")
+			(net 55 "MOT1")
 		)
 		(pad "87" smd roundrect
@@
 			(layers "F.Cu" "F.Mask" "F.Paste")
 			(roundrect_rratio 0.25)
-			(net 31 "GPS1_RX")
+			(net 56 "MOT2")
 		)
 		(pad "88" smd roundrect
@@
 			(layers "F.Cu" "F.Mask" "F.Paste")
 			(roundrect_rratio 0.25)
-			(net 77 "SPI1_MOSI")
+			(net 34 "HEATER_PWM")
 		)
 		(pad "89" smd roundrect
@@
 			(layers "F.Cu" "F.Mask" "F.Paste")
 			(roundrect_rratio 0.25)
-			(net 84 "SPI3_SCK")
+			(net 57 "MOT3")
 		)
 		(pad "90" smd roundrect
@@
 			(layers "F.Cu" "F.Mask" "F.Paste")
 			(roundrect_rratio 0.25)
-			(net 82 "SPI3_MISO")
+			(net 58 "MOT4")
 		)
 		(pad "91" smd roundrect
@@
 			(layers "F.Cu" "F.Mask" "F.Paste")
 			(roundrect_rratio 0.25)
-			(net 83 "SPI3_MOSI")
+			(net 59 "MOT5")
 		)
 		(pad "92" smd roundrect
@@
 			(layers "F.Cu" "F.Mask" "F.Paste")
 			(roundrect_rratio 0.25)
-			(net 37 "I2C1_SCL")
+			(net 60 "MOT6")
 		)
 		(pad "93" smd roundrect
@@
 			(layers "F.Cu" "F.Mask" "F.Paste")
 			(roundrect_rratio 0.25)
-			(net 38 "I2C1_SDA")
+			(net 61 "MOT7")
 		)
 		(pad "94" smd roundrect
@@
 			(layers "F.Cu" "F.Mask" "F.Paste")
 			(roundrect_rratio 0.25)
+			(net 62 "MOT8")
 		)
 		(pad "96" smd roundrect

Commit message: hw: R4 FEASIBLE re-mux — SKiDL source propagated (master 2026-05-22)
After AF verification killed the original 16-swap re-mux (10 INVALID
on LQFP-100), master directed: keep only feasible swaps + accept
SPI3/I2C1 stay on N + MOTs stay scattered (8-MOT-on-N impossible).

The feasible re-mux is 3 pin swaps (3-way shuffle):
1. SPI1_MOSI: pin 88 (PD7) → pin 31 (PA7) — AF5 ✓
2. HEATER_PWM: pin 31 (PA7) → pin 77 (PA15) — TIM2_CH1 AF1 ✓
3. BUZZER: pin 77 (PA15) → pin 88 (PD7) — plain GPIO ✓

Applied at both layers (source of truth + PCB):
- PCB: remux_pcb.py (2 swaps to achieve 3-way shuffle)
- SKiDL: imu_3c.py (SPI1_MOSI: PD7→PA7), power_3b.py (HEATER_PWM:
  PA7→PA15), gps_mag_3e.py (BUZZER: PA15→PD7)

SKiDL re-run: novapcb.net regenerated. 0 errors, 274 warnings
(existing baseline, not new). Netlist + PCB now agree.

Placement v13 unchanged (the geometry). Sensor island stays on S; the
S-island SPI3/I2C1 traces will route ~30mm MCU-N→island-S, accepted
as LQFP-100 pin-mux reality.

Next: Freerouting on the VALID netlist + v13 placement. Master's gate.

Co-Authored-By: Claude Opus 4.7 <noreply@anthropic.com>
Connections:
- U1 pad 22: (no net) -> MOT3
- U1 pad 23: (no net) -> MOT4
- U1 pad 24: (no net) -> MOT5
- U1 pad 25: (no net) -> MOT6
- U1 pad 28: SPI3_SCK -> (no net)
- U1 pad 32: SPI3_MISO -> (no net)
- U1 pad 33: SPI3_MOSI -> (no net)
- U1 pad 34: (no net) -> MOT1
- U1 pad 35: (no net) -> MOT2
- U1 pad 36: I2C1_SCL -> (no net)
- U1 pad 37: I2C1_SDA -> (no net)
- U1 pad 57: GPS1_TX -> (no net)
- U1 pad 58: GPS1_RX -> (no net)
- U1 pad 59: (no net) -> MOT7
- U1 pad 60: (no net) -> MOT8
- U1 pad 77: BUZZER -> HEATER_PWM
- U1 pad 86: MOT1 -> GPS1_TX
- U1 pad 87: MOT2 -> GPS1_RX
- U1 pad 88: HEATER_PWM -> BUZZER
- U1 pad 89: MOT3 -> SPI3_SCK
- U1 pad 90: MOT4 -> SPI3_MISO
- U1 pad 91: MOT5 -> SPI3_MOSI
- U1 pad 92: MOT6 -> I2C1_SCL
- U1 pad 93: MOT7 -> I2C1_SDA
- U1 pad 95: MOT8 -> (no net)
Changed lines of the file:
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@@
 			(layers "F.Cu" "F.Mask" "F.Paste")
 			(roundrect_rratio 0.25)
+			(net 57 "MOT3")
 		)
 		(pad "23" smd roundrect
@@
 			(layers "F.Cu" "F.Mask" "F.Paste")
 			(roundrect_rratio 0.25)
+			(net 58 "MOT4")
 		)
 		(pad "24" smd roundrect
@@
 			(layers "F.Cu" "F.Mask" "F.Paste")
 			(roundrect_rratio 0.25)
+			(net 59 "MOT5")
 		)
 		(pad "25" smd roundrect
@@
 			(layers "F.Cu" "F.Mask" "F.Paste")
 			(roundrect_rratio 0.25)
+			(net 60 "MOT6")
 		)
 		(pad "26" smd roundrect
@@
 			(layers "F.Cu" "F.Mask" "F.Paste")
 			(roundrect_rratio 0.25)
-			(net 84 "SPI3_SCK")
 		)
 		(pad "29" smd roundrect
@@
 			(layers "F.Cu" "F.Mask" "F.Paste")
 			(roundrect_rratio 0.25)
-			(net 82 "SPI3_MISO")
 		)
 		(pad "33" smd roundrect
@@
 			(layers "F.Cu" "F.Mask" "F.Paste")
 			(roundrect_rratio 0.25)
-			(net 83 "SPI3_MOSI")
 		)
 		(pad "34" smd roundrect
@@
 			(layers "F.Cu" "F.Mask" "F.Paste")
 			(roundrect_rratio 0.25)
+			(net 55 "MOT1")
 		)
 		(pad "35" smd roundrect
@@
 			(layers "F.Cu" "F.Mask" "F.Paste")
 			(roundrect_rratio 0.25)
+			(net 56 "MOT2")
 		)
 		(pad "36" smd roundrect
@@
 			(layers "F.Cu" "F.Mask" "F.Paste")
 			(roundrect_rratio 0.25)
-			(net 37 "I2C1_SCL")
 		)
 		(pad "37" smd roundrect
@@
 			(layers "F.Cu" "F.Mask" "F.Paste")
 			(roundrect_rratio 0.25)
-			(net 38 "I2C1_SDA")
 		)
 		(pad "38" smd roundrect
@@
 			(layers "F.Cu" "F.Mask" "F.Paste")
 			(roundrect_rratio 0.25)
-			(net 32 "GPS1_TX")
 		)
 		(pad "58" smd roundrect
@@
 			(layers "F.Cu" "F.Mask" "F.Paste")
 			(roundrect_rratio 0.25)
-			(net 31 "GPS1_RX")
 		)
 		(pad "59" smd roundrect
@@
 			(layers "F.Cu" "F.Mask" "F.Paste")
 			(roundrect_rratio 0.25)
+			(net 61 "MOT7")
 		)
 		(pad "60" smd roundrect
@@
 			(layers "F.Cu" "F.Mask" "F.Paste")
 			(roundrect_rratio 0.25)
+			(net 62 "MOT8")
 		)
 		(pad "61" smd roundrect
@@
 			(layers "F.Cu" "F.Mask" "F.Paste")
 			(roundrect_rratio 0.25)
-			(net 17 "BUZZER")
+			(net 34 "HEATER_PWM")
 		)
 		(pad "78" smd roundrect
@@
 			(layers "F.Cu" "F.Mask" "F.Paste")
 			(roundrect_rratio 0.25)
-			(net 55 "MOT1")
+			(net 32 "GPS1_TX")
 		)
 		(pad "87" smd roundrect
@@
 			(layers "F.Cu" "F.Mask" "F.Paste")
 			(roundrect_rratio 0.25)
-			(net 56 "MOT2")
+			(net 31 "GPS1_RX")
 		)
 		(pad "88" smd roundrect
@@
 			(layers "F.Cu" "F.Mask" "F.Paste")
 			(roundrect_rratio 0.25)
-			(net 34 "HEATER_PWM")
+			(net 17 "BUZZER")
 		)
 		(pad "89" smd roundrect
@@
 			(layers "F.Cu" "F.Mask" "F.Paste")
 			(roundrect_rratio 0.25)
-			(net 57 "MOT3")
+			(net 84 "SPI3_SCK")
 		)
 		(pad "90" smd roundrect
@@
 			(layers "F.Cu" "F.Mask" "F.Paste")
 			(roundrect_rratio 0.25)
-			(net 58 "MOT4")
+			(net 82 "SPI3_MISO")
 		)
 		(pad "91" smd roundrect
@@
 			(layers "F.Cu" "F.Mask" "F.Paste")
 			(roundrect_rratio 0.25)
-			(net 59 "MOT5")
+			(net 83 "SPI3_MOSI")
 		)
 		(pad "92" smd roundrect
@@
 			(layers "F.Cu" "F.Mask" "F.Paste")
 			(roundrect_rratio 0.25)
-			(net 60 "MOT6")
+			(net 37 "I2C1_SCL")
 		)
 		(pad "93" smd roundrect
@@
 			(layers "F.Cu" "F.Mask" "F.Paste")
 			(roundrect_rratio 0.25)
-			(net 61 "MOT7")
+			(net 38 "I2C1_SDA")
 		)
 		(pad "94" smd roundrect
@@
 			(layers "F.Cu" "F.Mask" "F.Paste")
 			(roundrect_rratio 0.25)
-			(net 62 "MOT8")
 		)
 		(pad "96" smd roundrect
